File: Kicad/Protoboard/auto.sch (KiCad schematic (older format))
At the start: 21 parts

Commit message: todo mas o menos ok
Parts:
- removed R?: 4k7, symbol R
- added D?: POWER, symbol LED
- added DS?: LCD-016N002L, WC1602A, symbol LCD-016N002L
- added R? (x5): 470, symbol R
- added SW? (x3): RESET, symbol SW_PUSH
Connections:
- net labels added: BTN1, BTN2, BTN3, BTN4, blink
- net labels removed: RA4
- wire segments 117 -> 126
Other:
- moved on the sheet: C?, D?, K?, P?, R?, SW?, U?
